Commit message: /tools vel change

File: tools/car_control/src/robot_description/urdf/target.urdf (robot description, URDF)
Before this commit: robot vlm_rl_arm, 10 links, 9 joints
Links:
- link base_link: mass 1.0 -> 7.925585093654501e-07; geometry collision mesh filename=package://robot_description/meshes/base_link.stl scale=0.001 0.001 0.001; visual mesh filename=package://robot_description/meshes/base_link.stl scale=0.001 0.001 0.001
- link base_link2_v2_1: mass 0.8 -> 0.8724221516717809; geometry collision mesh filename=package://robot_description/meshes/base_link2_v2_1.stl scale=0.001 0.001 0.001; visual mesh filename=package://robot_description/meshes/base_link2_v2_1.stl scale=0.001 0.001 0.001
- link base_link_2_1: mass 0.6 -> 1.6067306789990348; geometry collision mesh filename=package://robot_description/meshes/base_link_2_1.stl scale=0.001 0.001 0.001; visual mesh filename=package://robot_description/meshes/base_link_2_1.stl scale=0.001 0.001 0.001
- link camera_1: mass 0.1 -> 0.4003499999999954; geometry collision mesh filename=package://robot_description/meshes/camera_1.stl scale=0.001 0.001 0.001; visual mesh filename=package://robot_description/meshes/camera_1.stl scale=0.001 0.001 0.001
- link link3_mid_1: mass 0.05 -> 0.004162937218344747; geometry collision mesh filename=package://robot_description/meshes/link3_mid_1.stl scale=0.001 0.001 0.001; visual mesh filename=package://robot_description/meshes/link3_mid_1.stl scale=0.001 0.001 0.001
- link link3_v1_1: mass 1.0 -> 1.7894494256516058; geometry collision mesh filename=package://robot_description/meshes/link3_v1_1.stl scale=0.001 0.001 0.001; visual mesh filename=package://robot_description/meshes/link3_v1_1.stl scale=0.001 0.001 0.001
- link link4_v1_1: mass 0.9 -> 2.6308677332376194; geometry collision mesh filename=package://robot_description/meshes/link4_v1_1.stl scale=0.001 0.001 0.001; visual mesh filename=package://robot_description/meshes/link4_v1_1.stl scale=0.001 0.001 0.001
- link robot_ver7_grap1_2_v1_1: mass 0.1 -> 0.040626783640931655; geometry collision mesh filename=package://robot_description/meshes/robot_ver7_grap1_2_v1_1.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 scale=0.001 0.001 0.001; visual mesh filename=package://robot_description/meshes/robot_ver7_grap1_2_v1_1.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 scale=0.001 0.001 0.001
- link robot_ver7_grap2_2_v1_1: mass 0.1 -> 0.04062678364092949; geometry collision mesh filename=package://robot_description/meshes/robot_ver7_grap2_2_v1_1.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 scale=0.001 0.001 0.001; visual mesh filename=package://robot_description/meshes/robot_ver7_grap2_2_v1_1.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 scale=0.001 0.001 0.001
- link robot_ver7_link_4_v1_1: mass 0.4 -> 0.1836674229836172; geometry collision mesh filename=package://robot_description/meshes/robot_ver7_link_4_v1_1.s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 scale=0.001 0.001 0.001; visual mesh filename=package://robot_description/meshes/robot_ver7_link_4_v1_1.s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 scale=0.001 0.001 0.001

Commit message: arm smoothly move

File: tools/car_control/src/robot_description/urdf/target.urdf (robot description, URDF)
Before this commit: robot angle_excurate_arm_ver2, 10 links, 9 joints
Joints:
- joint Revolute 3: limit lower=0.0 upper=2.617994 effort=100 velocity=100 -> lower=0.0 upper=3.141593 effort=100 velocity=100
